File: designs/clock/clock.sch (KiCad schematic (older format))
At the start: 87 parts, among them J1 Conn_01x02_Power, J2 Conn_01x08, J3 Conn_01x08, J4 Conn_01x08, J5 Conn_01x08, Q1 BC547, Q10 2N7000, Q11 2N7000, Q12 2N7000, Q13 2N7000, Q14 2N7000, Q15 2N7000, Q16 2N7000, Q17 2N7000, Q18 2N7000, Q19 2N7000, Q2 BC547, Q20 2N7000, Q21 2N7000, Q22 2N7000, Q23 2N7000, Q24 2N7000, Q25 2N7000, Q26 2N7000, Q27 2N7000, Q28 2N7000, Q29 2N7000, Q3 2N7000, Q30 2N7000, Q31 2N7000, Q32 2N7000, Q33 2N7000, Q34 2N7000, Q35 2N7000, Q36 2N7000, Q37 2N7000, Q38 2N7000, Q39 2N7000, Q4 2N7000, Q40 2N7000, Q41 2N7000, Q42 2N7000, Q43 2N7000, Q44 2N7000, Q45 2N7000, Q46 2N7000, Q47 2N7000, Q48 2N7000, Q49 2N7000, Q5 2N7000, Q50 2N7000, Q6 2N7000, Q7 2N7000, Q8 2N7000, Q9 2N7000, SW1 SW_Push, SW2 SW_SPDT, SW3 SW_SPST, SW4 SW_Push

Commit message: Updated clock design.
Parts:
- added D101, D102: 1N4148, footprints:D_default, symbol 1N4148
- added R101, R102: 1k, footprints:R_small, symbol R
Connections:
- net Automatic_BaseClock: now also D101.1 (K), R101.2; no longer C1.1, R1.2
- net Automatic_BaseClock_Inv: now also D102.1 (K), R102.2; no longer C2.2, R4.2
- net GND: now also Q1.3 (E), Q17.1 (S), Q18.1 (S), Q2.3 (E), Q29.1 (S), Q30.1 (S), Q35.1 (S), Q36.1 (S), Q39.1 (S), Q40.1 (S), Q41.1 (S), Q44.1 (S)
- net VCC: now also R1.1, R10.1, R11.1, R12.1, R13.1, R14.1, R15.1, R20.1, R21.1, R4.1, RV1.1, R101.1, R102.1
- new net: C1.1, D101.2 (A), R1.2
- new net: C2.2, D102.2 (A), R4.2
Other:
- moved on the sheet: C1, C2, Q1, Q2, Q3, R1, R2, R3, R4, R5, R6, RV1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
