File: designs/memory/eprom/eprom.kicad_pcb (KiCad board)
At the start: 2 copper layers, 100 x 100 mm, 118 parts, among them J101 cardedge, Q101 2N7000, Q102 2N7000, Q103 2N7000, Q104 2N7000, Q105 2N7000, Q106 2N7000, Q107 2N7000, Q108 2N7000, Q109 2N7000, Q110 2N7000, Q111 2N7000, Q112 2N7000, Q113 2N7000, Q114 2N7000, Q115 2N7000, Q116 2N7000, Q117 2N7000, Q118 2N7000, Q201 2N7000, Q301 2N7000, Q401 2N7000, Q501 2N7000, Q601 2N7000, Q701 2N7000, Q801 2N7000, Q901 2N7000, SW201 DIPx08, SW301 DIPx08, SW401 DIPx08, SW501 DIPx08, SW601 DIPx08, SW701 DIPx08, SW801 DIPx08, SW901 DIPx08

Commit message: Latest design work updates.
Routing:
- net VCC: track 228.0 -> 230.2 mm
Changed lines of the file:
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@@
     (links 284)
     (no_connects 0)
-    (area 41.364999 15.329999 141.515001 115.480001)
+    (area 40.9575 14.605 141.922501 119.0175)
     (thickness 1.6)
     (drawings 6)
-    (tracks 755)
+    (tracks 759)
     (zones 0)
     (modules 118)
@@
   (segment (start 66.589258 62.189666) (end 66.589258 60.919666) (width 0.25) (layer F.Cu) (net 68))
   (segment (start 66.589258 60.919666) (end 67.859258 59.649666) (width 0.25) (layer F.Cu) (net 68))
+  (segment (start 48.895 106.68) (end 49.6625 106.68) (width 0.5) (layer F.Cu) (net 69))
+  (segment (start 48.895 106.68) (end 48.895 107.4375) (width 0.5) (layer F.Cu) (net 69))
+  (segment (start 48.1375 106.68) (end 48.895 106.68) (width 0.5) (layer F.Cu) (net 69))
+  (segment (start 48.895 107.4375) (end 48.9 107.4425) (width 0.5) (layer F.Cu) (net 69))
   (segment (start 88.5825 93.345) (end 89.2175 93.98) (width 0.5) (layer F.Cu) (net 69))
   (segment (start 88.5825 91.1225) (end 88.5825 93.345) (width 0.5) (layer F.Cu) (net 69))
